File: eagle/kelvin_1wire_B.brd (EAGLE design)
At the start: 72 x 42 mm, 46 parts, among them IC1 PIC18F2580, IC3 MCP2551SN, IC4 LM2575S, J1 OSTTE-12, J2 A00-108-220-450, Q1 10 MHz

Commit message: I/O handling in place
Connections:
- net T1: now also C13.1, R16.1; no longer C10.1, R7.1
- net T2: now also C12.1, R14.1; no longer C11.1, R12.1
- net T3: now also C11.1, R12.1; no longer C12.1, R14.1
- net T4: now also C10.1, R7.1; no longer C13.1, R16.1
Routing:
- net T1: track 38.7 -> 2.15 mm, vias 2 -> 0
- net T3: track 35.6 -> 0.00 mm, vias 2 -> 0
- net T4: track 27.6 -> 60.3 mm, vias 2 -> 4
- net T2: track 32.9 -> 63.8 mm, vias 2 -> 4
Changed lines of the file:
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@@
 <via x="40.64" y="10.16" extent="1-16" drill="0.3556"/>
 </signal>
-<signal name="T1">
-<contactref element="IC1" pad="14"/>
+<signal name="N$9">
+<contactref element="C14" pad="2"/>
+<contactref element="IC1" pad="6"/>
+<wire x1="41.82" y1="29.585" x2="54.96" y2="30.62" width="0" layer="19" extent="1-1"/>
+</signal>
+<signal name="T4">
 <contactref element="R7" pad="1"/>
 <contactref element="C10" pad="1"/>
 <wire x1="14.2" y1="28.94" x2="14.2" y2="30.48" width="0.254" layer="1"/>
 <wire x1="14.15" y1="28.89" x2="14.2" y2="28.94" width="0.254" layer="1"/>
-<wire x1="41.82" y1="39.745" x2="39.445" y2="39.745" width="0.254" layer="1"/>
 <wire x1="39.445" y1="39.745" x2="39.1" y2="39.4" width="0.254" layer="1"/>
 <via x="39.1" y="39.4" extent="1-16" drill="0.6" shape="square"/>
@@
 <wire x1="15.9" y1="30.5" x2="14.22" y2="30.5" width="0.254" layer="1"/>
 <wire x1="14.22" y1="30.5" x2="14.2" y2="30.48" width="0.254" layer="1"/>
+<contactref element="IC1" pad="18"/>
+<wire x1="31.66" y1="35.935" x2="29.965" y2="35.935" width="0.254" layer="1"/>
+<wire x1="29.965" y1="35.935" x2="29.9" y2="36" width="0.254" layer="1"/>
+<via x="29.9" y="36" extent="1-16" drill="0.6" shape="square"/>
+<wire x1="29.9" y1="36" x2="28.6" y2="36" width="0.254" layer="16"/>
+<wire x1="28.6" y1="36" x2="28" y2="35.4" width="0.254" layer="16"/>
+<wire x1="28" y1="35.4" x2="28" y2="27.9" width="0.254" layer="16"/>
+<wire x1="28" y1="27.9" x2="24.5" y2="24.4" width="0.254" layer="16"/>
+<wire x1="24.5" y1="24.4" x2="24.5" y2="17.6" width="0.254" layer="16"/>
+<wire x1="24.5" y1="17.6" x2="24" y2="17.1" width="0.254" layer="16"/>
+<via x="24" y="17.1" extent="1-16" drill="0.6" shape="square"/>
+<wire x1="31.66" y1="35.935" x2="34.4" y2="39.4" width="0" layer="19" extent="1-16"/>
+</signal>
+<signal name="T1">
+<contactref element="R16" pad="1"/>
+<contactref element="C13" pad="1"/>
+<wire x1="22.4" y1="17.09" x2="22.4" y2="14.95" width="0.254" layer="1"/>
+<wire x1="22.41" y1="17.1" x2="22.4" y2="17.09" width="0.254" layer="1"/>
+<contactref element="IC1" pad="14"/>
+<wire x1="22.41" y1="17.1" x2="41.82" y2="39.745" width="0" layer="19" extent="1-1"/>
 </signal>
 <signal name="T2">
+<contactref element="R14" pad="1"/>
+<contactref element="C12" pad="1"/>
+<wire x1="14.89" y1="17.29" x2="14.7" y2="18.81" width="0.254" layer="1"/>
+<wire x1="14.85" y1="16.71" x2="14.89" y2="17.29" width="0.254" layer="1"/>
+<wire x1="14.82" y1="16.75" x2="14.85" y2="16.71" width="0.254" layer="1"/>
+<wire x1="14.65" y1="16.94" x2="14.82" y2="16.75" width="0.254" layer="1"/>
+<wire x1="27.795" y1="37.205" x2="27.7" y2="37.3" width="0.254" layer="1"/>
+<via x="27.7" y="37.3" extent="1-16" drill="0.6" shape="square"/>
+<wire x1="27.7" y1="37.3" x2="27" y2="37.3" width="0.254" layer="16"/>
+<wire x1="27" y1="37.3" x2="25.8" y2="36.1" width="0.254" layer="16"/>
+<wire x1="25.8" y1="36.1" x2="25.8" y2="27.7" width="0.254" layer="16"/>
+<wire x1="25.8" y1="27.7" x2="23.9" y2="25.8" width="0.254" layer="16"/>
+<wire x1="23.9" y1="25.8" x2="17.5" y2="25.8" width="0.254" layer="16"/>
+<wire x1="17.5" y1="25.8" x2="17.3" y2="25.6" width="0.254" layer="16"/>
+<wire x1="17.3" y1="25.6" x2="17.3" y2="19.5" width="0.254" layer="16"/>
+<wire x1="17.3" y1="19.5" x2="16.6" y2="18.8" width="0.254" layer="16"/>
+<via x="16.6" y="18.8" extent="1-16" drill="0.6" shape="square"/>
+<wire x1="16.6" y1="18.8" x2="14.71" y2="18.8" width="0.254" layer="1"/>
+<wire x1="14.71" y1="18.8" x2="14.7" y2="18.81" width="0.254" layer="1"/>
 <contactref element="IC1" pad="15"/>
-<contactref element="R12" pad="1"/>
-<contactref element="C11" pad="1"/>
 <wire x1="14.51" y1="22.24" x2="14.51" y2="23.3" width="0.254" layer="1"/>
-<wire x1="14.51" y1="23.3" x2="14.51" y2="23.8" width="0.254" layer="1"/>
-<wire x1="14.32" y1="22.05" x2="14.51" y2="22.24" width="0.254" layer="1"/>
 <wire x1="31.66" y1="39.745" x2="28.145" y2="39.745" width="0.254" layer="1"/>
 <wire x1="28.145" y1="39.745" x2="27.7" y2="39.3" width="0.254" layer="1"/>
@@
 <wire x1="16.2" y1="23.7" x2="14.91" y2="23.7" width="0.254" layer="1"/>
 <wire x1="14.91" y1="23.7" x2="14.51" y2="23.3" width="0.254" layer="1"/>
+<wire x1="25.8" y1="27.7" x2="24.8" y2="28.2" width="0" layer="19" extent="16-16"/>
 </signal>
 <signal name="T3">
 <contactref element="IC1" pad="17"/>
-<contactref element="R14" pad="1"/>
-<contactref element="C12" pad="1"/>
-<wire x1="14.89" y1="17.29" x2="14.7" y2="18.81" width="0.254" layer="1"/>
-<wire x1="14.85" y1="16.71" x2="14.89" y2="17.29" width="0.254" layer="1"/>
-<wire x1="14.82" y1="16.75" x2="14.85" y2="16.71" width="0.254" layer="1"/>
-<wire x1="14.65" y1="16.94" x2="14.82" y2="16.75" width="0.254" layer="1"/>
-<wire x1="31.66" y1="37.205" x2="27.795" y2="37.205" width="0.254" layer="1"/>
-<wire x1="27.795" y1="37.205" x2="27.7" y2="37.3" width="0.254" layer="1"/>
-<via x="27.7" y="37.3" extent="1-16" drill="0.6" shape="square"/>
-<wire x1="27.7" y1="37.3" x2="27" y2="37.3" width="0.254" layer="16"/>
-<wire x1="27" y1="37.3" x2="25.8" y2="36.1" width="0.254" layer="16"/>
-<wire x1="25.8" y1="36.1" x2="25.8" y2="27.7" width="0.254" layer="16"/>
-<wire x1="25.8" y1="27.7" x2="23.9" y2="25.8" width="0.254" layer="16"/>
-<wire x1="23.9" y1="25.8" x2="17.5" y2="25.8" width="0.254" layer="16"/>
-<wire x1="17.5" y1="25.8" x2="17.3" y2="25.6" width="0.254" layer="16"/>
-<wire x1="17.3" y1="25.6" x2="17.3" y2="19.5" width="0.254" layer="16"/>
-<wire x1="17.3" y1="19.5" x2="16.6" y2="18.8" width="0.254" layer="16"/>
-<via x="16.6" y="18.8" extent="1-16" drill="0.6" shape="square"/>
-<wire x1="16.6" y1="18.8" x2="14.71" y2="18.8" width="0.254" layer="1"/>
-<wire x1="14.71" y1="18.8" x2="14.7" y2="18.81" width="0.254" layer="1"/>
-</signal>
-<signal name="T4">
-<contactref element="IC1" pad="18"/>
-<contactref element="R16" pad="1"/>
-<contactref element="C13" pad="1"/>
-<wire x1="22.4" y1="17.09" x2="22.4" y2="14.95" width="0.254" layer="1"/>
-<wire x1="22.41" y1="17.1" x2="22.4" y2="17.09" width="0.254" layer="1"/>
-<wire x1="31.66" y1="35.935" x2="29.965" y2="35.935" width="0.254" layer="1"/>
-<wire x1="29.965" y1="35.935" x2="29.9" y2="36" width="0.254" layer="1"/>
-<via x="29.9" y="36" extent="1-16" drill="0.6" shape="square"/>
-<wire x1="29.9" y1="36" x2="28.6" y2="36" width="0.254" layer="16"/>
-<wire x1="28.6" y1="36" x2="28" y2="35.4" width="0.254" layer="16"/>
-<wire x1="28" y1="35.4" x2="28" y2="27.9" width="0.254" layer="16"/>
-<wire x1="28" y1="27.9" x2="24.5" y2="24.4" width="0.254" layer="16"/>
-<wire x1="24.5" y1="24.4" x2="24.5" y2="17.6" width="0.254" layer="16"/>
-<wire x1="24.5" y1="17.6" x2="24" y2="17.1" width="0.254" layer="16"/>
-<via x="24" y="17.1" extent="1-16" drill="0.6" shape="square"/>
-<wire x1="24" y1="17.1" x2="22.41" y2="17.1" width="0.254" layer="1"/>
-</signal>
-<signal name="N$9">
-<contactref element="C14" pad="2"/>
-<contactref element="IC1" pad="6"/>
-<wire x1="41.82" y1="29.585" x2="54.96" y2="30.62" width="0" layer="19" extent="1-1"/>
+<contactref element="R12" pad="1"/>
+<contactref element="C11" pad="1"/>
+<wire x1="14.51" y1="23.8" x2="31.66" y2="37.205" width="0" layer="19" extent="1-1"/>
+<wire x1="14.32" y1="22.05" x2="14.51" y2="23.8" width="0" layer="19" extent="1-1"/>
 </signal>
 </signals>
